File: boards/esp8266/mymote-esp8266.brd (EAGLE design)
At the start: 44.5 x 33.2 mm, 36 parts, among them IC1 ESP-12-SMD, IC31 MCP73831/OT, IC32 MCP1703CB

Commit message: Relay board and oter small changes
Parts:
- removed C35: 100nF, xose:0805
- added D1: 1N5819, xose:0805_DIODE
- added Q1: (no value), xose:SOT23-WIDE
- added R7: 2K, xose:0805
- added SJ1: SWITCH, xose:SJ_2S-TRACE-PTH
- C34: value 10uF -> 1uF
- IC32: value MCP1703CB -> AP2112-3V3; device xose:SOT23 -> xose:SOT23-5L
- SJ21, SJ22, SJ23, SJ24: value (none) -> SOLDERJUMPERNO
- moved C34 7.24 mm to (38.4, 8.26), turned to 90 degrees
- moved C33 5.85 mm to (35.9, 8.26), turned to 90 degrees
- moved IC32 3.84 mm to (33.3, 7.62), turned to 180 degrees
Connections:
- new net N$9: D1.C, Q1.2, SJ1.1
- new net VIN: C33.1, IC32.1, IC32.3, SJ1.2
- net 3V3: now also IC32.5; no longer C35.1, IC32.2
- net GND: now also IC32.2, R7.2; no longer C35.2, IC32.1
- net VBAT: now also Q1.3; no longer C33.1, IC32.3
- net VSOL: now also D1.A, Q1.1, R7.1
