File: boards/core/mymote-core.brd (EAGLE design)
At the start: 44.5 x 33.2 mm, 38 parts, among them IC1 ATMEGA328P-AU-TQFP32, IC2 MCP73831/OT, IC3 MCP1703CB, IC4 AT25F512BWIDE_5.3MM

Commit message: Relay board and oter small changes
Parts:
- added U$4: RFM69CW-MINPADS, xose:RFM69CW-MINPADS
- U$3: value RFM69C&9X -> RFM69HCW-RFM95; device xose:RFM69&9X -> xose:RFM69HCW-RFM95-MINPADS
- moved SJ2 0.52 mm to (7.37, 8.38), turned to 180 degrees
- moved U$1 0.13 mm to (5.21, 8.38)
Connections:
- net 3V3: now also U$4.2
- net ANT: now also U$4.1
- net D10_SS: now also U$4.6
- net D11_MOSI: now also U$4.4
- net D12_MISO: now also U$4.7
- net D13_SCK: now also U$4.5
- net D2: now also U$4.8
- net GND: now also U$3.GND1, U$3.GND2, U$4.3, U$4.9
Routing:
- net D12_MISO: track 24.7 -> 53.9 mm, vias 1 -> 5
- net ANT: track 7.17 -> 33.9 mm, vias 0 -> 3
- net GND: track 35.3 -> 45.9 mm, vias 15 -> 16
- net D13_SCK: track 26.1 -> 36.0 mm, vias 4 -> 5
- net D2: track 28.0 -> 36.2 mm
- net D10_SS: track 18.9 -> 24.9 mm
- net D8: track 15.1 -> 18.2 mm
- net D11_MOSI: track 35.6 -> 38.7 mm
- net VIN: track 32.0 -> 33.2 mm
- net N$9: track 17.5 -> 18.5 mm
- net D5: track 7.98 -> 8.79 mm
- net N$8: track 3.03 -> 3.75 mm
- net D4: track 15.4 -> 16.0 mm
- net D9: track 9.63 -> 9.05 mm, vias 0 -> 1
- net RST: track 31.1 -> 31.7 mm
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Other:
- outline, holes or cut-outs redrawn
- board text added: "Tinkerman 2017 MYMOTE CORE v0.2.20170617"
- board text removed: "Tinkerman 2017 MYMOTE CORE v0.2.20170604"

Commit message: Update
Connections:
- removed net N$6: C10.1, C9.2
- net RST: now also C10.1, C9.2
Routing:
- net RST: track 31.7 -> 35.6 mm
- net N$6: track 3.03 -> 0.00 mm
Other:
- board text added: "Tinkerman 2018 MYMOTE CORE v0.3.20180204"
- board text removed: "Tinkerman 2017 MYMOTE CORE v0.2.20170617"
Changed lines of the file:
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@@
 <?xml version="1.0" encoding="utf-8"?>
 <!DOCTYPE eagle SYSTEM "eagle.dtd">
-<eagle version="8.2.1">
+<eagle version="8.3.2">
 <drawing>
 <settings>
 <setting alwaysvectorfont="no"/>
+<setting keepoldvectorfont="yes"/>
 <setting verticaltext="up"/>
 </settings>
@@
 <layer number="27" name="tValues" color="7" fill="1" visible="no" active="yes"/>
 <layer number="28" name="bValues" color="7" fill="1" visible="no" active="yes"/>
-<layer number="29" name="tStop" color="7" fill="3" visible="no" active="yes"/>
-<layer number="30" name="bStop" color="7" fill="6" visible="no" active="yes"/>
+<layer number="29" name="tStop" color="7" fill="3" visible="yes" active="yes"/>
+<layer number="30" name="bStop" color="7" fill="6" visible="yes" active="yes"/>
 <layer number="31" name="tCream" color="12" fill="1" visible="no" active="yes"/>
 <layer number="32" name="bCream" color="7" fill="5" visible="no" active="yes"/>
@@
 <text x="31.75" y="20.574" size="0.762" layer="26" font="vector" ratio="18" rot="MR0" align="top-center">A0</text>
 <text x="16.51" y="2.54" size="0.762" layer="26" font="vector" ratio="18" rot="MR0" align="bottom-center">7</text>
-<text x="37.592" y="2.667" size="0.8128" layer="26" font="vector" ratio="15" rot="MR0" align="center">Tinkerman 2017
+<text x="37.592" y="2.667" size="0.8128" layer="26" font="vector" ratio="15" rot="MR0" align="center">Tinkerman 2018
 MYMOTE CORE
-v0.2.20170617</text>
+v0.3.20180204</text>
 <rectangle x1="39.4002" y1="4.7693" x2="39.451" y2="4.7947" layer="26" rot="R180"/>
 <rectangle x1="36.3014" y1="4.7693" x2="36.3522" y2="4.7947" layer="26" rot="R180"/>
@@
 <wire x1="1.651" y1="3.556" x2="1.397" y2="3.302" width="0.1524" layer="1"/>
 <wire x1="1.397" y1="3.302" x2="1.397" y2="1.397" width="0.1524" layer="1"/>
-<wire x1="9.652" y1="3.556" x2="1.651" y2="3.556" width="0.1524" layer="1"/>
+<wire x1="7.366" y1="3.556" x2="9.652" y2="3.556" width="0.1524" layer="1"/>
+<wire x1="7.366" y1="3.556" x2="1.651" y2="3.556" width="0.1524" layer="1"/>
 <wire x1="9.652" y1="3.556" x2="13.462" y2="3.556" width="0.1524" layer="1"/>
 <wire x1="17.634" y1="15.8496" x2="17.653" y2="15.8306" width="0.1524" layer="1"/>
@@
 <wire x1="13.208" y1="3.937" x2="13.208" y2="11.811" width="0.1524" layer="16"/>
 <wire x1="13.208" y1="11.811" x2="13.462" y2="12.065" width="0.1524" layer="16"/>
+<contactref element="C9" pad="2"/>
+<contactref element="C10" pad="1"/>
+<wire x1="5.08" y1="6.234" x2="6.88" y2="4.434" width="0.1524" layer="1"/>
+<wire x1="6.88" y1="4.434" x2="7.366" y2="4.434" width="0.1524" layer="1"/>
+<wire x1="7.366" y1="4.434" x2="7.366" y2="3.556" width="0.1524" layer="1"/>
 </signal>
 <signal name="D9">
@@
 <wire x1="34.036" y1="17.272" x2="34.036" y2="13.589" width="0.1524" layer="16"/>
 </signal>
-<signal name="N$6">
-<contactref element="C9" pad="2"/>
-<contactref element="C10" pad="1"/>
-<wire x1="5.08" y1="6.234" x2="6.88" y2="4.434" width="0.1524" layer="1"/>
-<wire x1="6.88" y1="4.434" x2="7.366" y2="4.434" width="0.1524" layer="1"/>
-</signal>
 </signals>
