File: boards/core/mymote-core.sch (EAGLE design)
At the start: 38 parts, among them IC1 ATMEGA328P-AU-TQFP32, IC2 MCP73831/OT, IC3 MCP1703CB, IC4 AT25F512BWIDE_5.3MM

Commit message: Relay board and oter small changes
Parts:
- added U$4: RFM69CW-MINPADS, xose:RFM69CW-MINPADS
- U$3: value RFM69C&9X -> RFM69HCW-RFM95; device xose:RFM69C&9X -> xose:RFM69HCW-RFM95
Connections:
- net 3V3: now also U$4.3.3V
- net ANT: now also U$4.ANT
- net D10_SS: now also U$4.NSS
- net D11_MOSI: now also U$4.MOSI
- net D12_MISO: now also U$4.MISO
- net D13_SCK: now also U$4.SCK
- net D2: now also U$4.DIO0
- net GND: now also U$3.GND1, U$3.GND2, U$4.GND@1, U$4.GND@2

Commit message: Update
Connections:
- removed net N$6: C10.1, C9.2
- net RST: now also C10.1, C9.2
Changed lines of the file:
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@@
 <?xml version="1.0" encoding="utf-8"?>
 <!DOCTYPE eagle SYSTEM "eagle.dtd">
-<eagle version="8.2.1">
+<eagle version="8.3.2">
 <drawing>
 <settings>
 <setting alwaysvectorfont="no"/>
+<setting keepoldvectorfont="yes"/>
 <setting verticaltext="up"/>
 </settings>
-<grid distance="0.05" unitdist="inch" unit="inch" style="lines" multiple="1" display="no" altdistance="0.01" altunitdist="inch" altunit="inch"/>
+<grid distance="0.1" unitdist="inch" unit="inch" style="lines" multiple="1" display="no" altdistance="0.01" altunitdist="inch" altunit="inch"/>
 <layers>
 <layer number="1" name="Top" color="4" fill="1" visible="no" active="no"/>
@@
 <attribute name="PROJECT_LICENSE" value="CC-SA-BY 3.0"/>
 <attribute name="PROJECT_NAME" value="MYMOTE - CORE"/>
-<attribute name="PROJECT_VERSION" value="0.2.20170617"/>
+<attribute name="PROJECT_VERSION" value="0.3.20180204"/>
 </attributes>
 <variantdefs>
@@
 <label x="182.88" y="168.91" size="1.778" layer="95"/>
 </segment>
+<segment>
+<pinref part="C9" gate="G$1" pin="2"/>
+<wire x1="203.2" y1="96.52" x2="205.74" y2="96.52" width="0.1524" layer="91"/>
+<label x="208.28" y="96.52" size="1.778" layer="95"/>
+<pinref part="C10" gate="G$1" pin="1"/>
+<wire x1="205.74" y1="96.52" x2="213.36" y2="96.52" width="0.1524" layer="91"/>
+<wire x1="205.74" y1="96.52" x2="205.74" y2="93.98" width="0.1524" layer="91"/>
+<junction x="205.74" y="96.52"/>
+</segment>
 </net>
 <net name="D9" class="0">
@@
 </segment>
 </net>
-<net name="N$6" class="0">
-<segment>
-<pinref part="C9" gate="G$1" pin="2"/>
-<wire x1="203.2" y1="96.52" x2="205.74" y2="96.52" width="0.1524" layer="91"/>
-<label x="208.28" y="96.52" size="1.778" layer="95"/>
-<pinref part="C10" gate="G$1" pin="1"/>
-<wire x1="205.74" y1="96.52" x2="213.36" y2="96.52" width="0.1524" layer="91"/>
-<wire x1="205.74" y1="96.52" x2="205.74" y2="93.98" width="0.1524" layer="91"/>
-<junction x="205.74" y="96.52"/>
-</segment>
-</net>
 </nets>
 </sheet>
@@
 <compatibility>
 <note version="8.2" severity="warning">
-Since Version 8.2, Eagle supports online libraries. The ids
+Since Version 8.2, EAGLE supports online libraries. The ids
 of those online libraries will not be understood (or retained)
 with this version.
