File: boards/logger/mymote-logger.brd (EAGLE design)
At the start: 33.3 x 33.2 mm, 15 parts, among them IC5 DS1337S+

Commit message: Update
Connections:
- net VBAT: no longer R1.1
- net VRTC: now also R1.1
Routing:
- net VRTC: track 8.52 -> 13.0 mm
- net VBAT: track 11.7 -> 10.3 mm
Other:
- board text added: "Tinkerman 2017 MYMOTE LOGGER v0.2.20171019"
- board text removed: "Tinkerman 2017 MYMOTE LOGGER v0.1.20170507"
Changed lines of the file:
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@@
 <?xml version="1.0" encoding="utf-8"?>
 <!DOCTYPE eagle SYSTEM "eagle.dtd">
-<eagle version="8.0.1">
+<eagle version="8.3.2">
 <drawing>
 <settings>
 <setting alwaysvectorfont="no"/>
+<setting keepoldvectorfont="yes"/>
 <setting verticaltext="up"/>
 </settings>
@@
 <text x="11.049" y="17.526" size="0.8128" layer="25" font="vector" ratio="15" rot="R180" align="center">Tinkerman 2017
 MYMOTE LOGGER
-v0.1.20170507</text>
+v0.2.20171019</text>
 <rectangle x1="4.4752" y1="14.9293" x2="4.526" y2="14.9547" layer="25" rot="R180"/>
 <rectangle x1="1.3764" y1="14.9293" x2="1.4272" y2="14.9547" layer="25" rot="R180"/>
@@
 <attribute name="OC_FARNELL" value="1379748" x="-22.733" y="6.35" size="1.778" layer="27" display="off"/>
 <attribute name="OC_NEWARK" value="08J6237" x="-22.733" y="6.35" size="1.778" layer="27" display="off"/>
+<attribute name="PACKAGE" value="SOIC-8" x="-22.733" y="6.35" size="1.778" layer="27" display="off"/>
 <attribute name="SUPPLIER" value="Maxim" x="-22.733" y="6.35" size="1.778" layer="27" display="off"/>
-<attribute name="PACKAGE" value="SOIC-8" x="-22.733" y="6.35" size="1.778" layer="27" display="off"/>
 </element>
 <element name="D1" library="xose" package="0805_DIODE" value="DIODE-SMD" x="6.985" y="13.462"/>
@@
 <signal name="VRTC">
 <contactref element="IC5" pad="8"/>
-<contactref element="D1" pad="C"/>
 <contactref element="Q2" pad="3"/>
 <wire x1="11.303" y1="8.4328" x2="11.4808" y2="8.255" width="0.1524" layer="1"/>
 <wire x1="11.303" y1="13.165" x2="11.303" y2="8.4328" width="0.1524" layer="1"/>
+<wire x1="11.006" y1="13.462" x2="11.303" y2="13.165" width="0.1524" layer="1"/>
+<contactref element="D1" pad="C"/>
+<contactref element="R1" pad="1"/>
 <wire x1="7.885" y1="13.462" x2="11.006" y2="13.462" width="0.1524" layer="1"/>
 <wire x1="11.006" y1="13.462" x2="11.303" y2="13.165" width="0.1524" layer="1"/>
+<wire x1="6.085" y1="10.922" x2="6.085" y2="11.927" width="0.1524" layer="1"/>
+<wire x1="6.085" y1="11.927" x2="6.35" y2="12.192" width="0.1524" layer="1"/>
+<wire x1="6.35" y1="12.192" x2="7.62" y2="12.192" width="0.1524" layer="1"/>
+<wire x1="7.62" y1="12.192" x2="7.874" y2="12.446" width="0.1524" layer="1"/>
+<wire x1="7.874" y1="12.446" x2="7.874" y2="13.451" width="0.1524" layer="1"/>
+<wire x1="7.874" y1="13.451" x2="7.885" y2="13.462" width="0.1524" layer="1"/>
 </signal>
 <signal name="N$10">
@@
 </signal>
 <signal name="VBAT">
+<contactref element="ANALOGSIDE" pad="12"/>
 <contactref element="D1" pad="A"/>
-<contactref element="R1" pad="1"/>
-<contactref element="ANALOGSIDE" pad="12"/>
-<wire x1="6.085" y1="10.922" x2="6.085" y2="13.462" width="0.1524" layer="1"/>
-<wire x1="6.085" y1="13.462" x2="3.937" y2="15.61" width="0.1524" layer="1"/>
-<wire x1="3.937" y1="15.61" x2="3.937" y2="21.717" width="0.1524" layer="1"/>
+<wire x1="3.937" y1="13.716" x2="4.191" y2="13.462" width="0.1524" layer="1"/>
+<wire x1="4.191" y1="13.462" x2="6.085" y2="13.462" width="0.1524" layer="1"/>
+<wire x1="3.937" y1="21.717" x2="3.937" y2="13.716" width="0.1524" layer="1"/>
 </signal>
 <signal name="N$14">
