File: boards/relay/mymote-relay.brd (EAGLE design)
At the start: 33.3 x 33.2 mm, 10 parts

Commit message: Update
Parts:
- removed D1: 1N4148, xose:SOD80
- removed Q1: (no value), xose:SOT23
- removed R1: 1K, xose:0805
- removed R2: 10K, xose:0805
- added IC1: LB1973JA, xose:SSOP16
- moved R3 0.57 mm to (2.41, 5.71), turned to 90 degrees
Connections:
- removed net N$4: D1.1, Q1.3, RLY1.COIL2
- removed net N$5: Q1.1, R1.2, R2.2
- new net N$2: IC1.12, RLY1.COIL1
- new net N$3: IC1.11, RLY1.COIL2
- net 3V3: now also IC1.1; no longer D1.2, RLY1.COIL1
- net D4: no longer R1.1
- net D8: now also IC1.6
- net D9: now also IC1.7
- net GND: now also IC1.9; no longer Q1.2, R2.1
Routing:
- net D9: track 0.00 -> 21.1 mm
- net D8: track 0.00 -> 20.3 mm
- net D4: track 12.9 -> 0.00 mm
- net N$4: track 10.4 -> 0.00 mm
- net N$5: track 8.17 -> 0.00 mm
- net N$2: track 0.00 -> 5.61 mm
- net GND: track 23.1 -> 28.3 mm
- net N$3: track 0.00 -> 4.33 mm
- net D3: track 12.6 -> 12.0 mm
- net 3V3: track 34.4 -> 34.0 mm, vias 1 -> 0
Other:
- outline, holes or cut-outs redrawn
- board text added: "Tinkerman 2017 MYMOTE RELAY v0.2.20170805"
- board text removed: "Tinkerman 2017 MYMOTE RELAY v0.1.20170705"
