File: boards/relay/mymote-relay.sch (EAGLE design)
At the start: 10 parts

Commit message: Update
Parts:
- removed D1: 1N4148, xose:DIODE
- removed Q1: (no value), xose:MOSFET-NREFLOW
- removed R1: 1K, xose:RESISTOR0805
- removed R2: 10K, xose:RESISTOR0805
- added IC1: LB1973JA, xose:LB1973JA
Connections:
- removed net N$4: D1.A, Q1.D, RLY1.COIL2
- removed net N$5: Q1.G, R1.2, R2.2
- new net N$2: IC1.OUT1, RLY1.COIL1
- new net N$3: IC1.OUT2, RLY1.COIL2
- net 3V3: now also IC1.VCC; no longer D1.C, RLY1.COIL1
- net D4: no longer R1.1
- net D8: now also IC1.IN1
- net D9: now also IC1.IN2
- net GND: now also IC1.GND; no longer Q1.S, R2.1
Other:
- note added: "BUTTON"
- moved on the sheet: JP1, JP3, R3, RLY1
